File: Building Resources/KiCad PCB Files/490 Power Supply Circuit.kicad_pcb (KiCad board)
At the start: 2 copper layers, 16 parts, among them J1 Screw_Terminal_01x10, U1 LM2596T-3.3, U3 ESP32-DEVKITC-32D

Commit message: Upload new KiCad Files.
Parts:
- added D2: RED, LED_THT:LED_D4.0mm, F.Cu at (67.7, 44.0)
- added D3: YELLOW, LED_THT:LED_D4.0mm, F.Cu at (67.7, 52.0)
- added D4: GREEN, LED_THT:LED_D4.0mm, F.Cu at (67.7, 60.5)
- added J10: 2319, TerminalBlock_4Ucon:TerminalBlock_4Ucon_1x02_P3.50mm_Vertical, F.Cu at (75.4, 125.8)
- added J11: 3.3/18, TerminalBlock_4Ucon:TerminalBlock_4Ucon_1x02_P3.50mm_Vertical, F.Cu at (75.1, 85.8)
- added J12: 0017, TerminalBlock_4Ucon:TerminalBlock_4Ucon_1x02_P3.50mm_Vertical, F.Cu at (75.0, 104.5)
- added J13: 0504, TerminalBlock_4Ucon:TerminalBlock_4Ucon_1x02_P3.50mm_Vertical, F.Cu at (199.1, 82.2)
- added J14: 0215, TerminalBlock_4Ucon:TerminalBlock_4Ucon_1x02_P3.50mm_Vertical, F.Cu at (75.0, 113.8)
- added J15: 1312, TerminalBlock_4Ucon:TerminalBlock_4Ucon_1x02_P3.50mm_Vertical, F.Cu at (199.1, 59.4)
- added J16: 14, TerminalBlock_4Ucon:TerminalBlock_4Ucon_1x02_P3.50mm_Vertical, F.Cu at (199.6, 70.2)
- added J2: 3.3V, TerminalBlock_4Ucon:TerminalBlock_4Ucon_1x02_P3.50mm_Vertical, F.Cu at (145.0, 41.4)
- added J3: 3.3V AND GND, TerminalBlock_4Ucon:TerminalBlock_4Ucon_1x02_P3.50mm_Vertical, F.Cu at (145.0, 51.4)
- added J4: GND, TerminalBlock_4Ucon:TerminalBlock_4Ucon_1x02_P3.50mm_Vertical, F.Cu at (145.0, 61.5)
- added J5: LED'S, TerminalBlock_4Ucon:TerminalBlock_4Ucon_1x02_P3.50mm_Vertical, F.Cu at (145.0, 81.0)
- added J6: LED'S AND GND, TerminalBlock_4Ucon:TerminalBlock_4Ucon_1x02_P3.50mm_Vertical, F.Cu at (145.0, 90.8)
- added J7: SPEAKER, TerminalBlock_4Ucon:TerminalBlock_4Ucon_1x02_P3.50mm_Vertical, F.Cu at (145.0, 71.3)
- added J8: VOLUME/JOHNS RST, TerminalBlock_4Ucon:TerminalBlock_4Ucon_1x02_P3.50mm_Vertical, F.Cu at (75.0, 95.0)
- added J9: 22/GND, TerminalBlock_4Ucon:TerminalBlock_4Ucon_1x02_P3.50mm_Vertical, F.Cu at (75.0, 76.5)
- added U2: DFR0299, DFR0299:DFR0299, F.Cu at (113.5, 75.5)
- C2: value 220uF -> 220u
- J1: value Screw_Terminal_01x10 -> BATTERY TERMS; footprint TerminalBlock:TerminalBlock_MaiXu_MX126-5.0-10P_1x10_P5.00mm -> TerminalBlock_4Ucon:TerminalBlock_4Ucon_1x02_P3.50mm_Vertical
- L1: value 68mh -> 68m
- moved J1 105.2 mm to (145.5, 31.5), turned to -90 degrees
- moved U3 72.7 mm to (111.0, 106.2), turned to -90 degrees
- moved R6 70.0 mm to (137.3, 84.0), turned to 180 degrees
- moved R7 70.0 mm to (137.3, 88.0), turned to 180 degrees
- moved R8 69.7 mm to (137.5, 80.0), turned to 180 degrees
- moved R2-2 65.7 mm to (123.0, 55.2), turned to -90 degrees
- moved R2-1 64.4 mm to (118.5, 47.2), turned to -90 degrees
- moved L1 63.2 mm to (131.5, 64.5), turned to 90 degrees
- moved R3 62.8 mm to (126.5, 40.2), turned to -90 degrees
- moved C2 53.6 mm to (135.0, 50.2), turned to 90 degrees
- moved R5 52.3 mm to (114.5, 47.0), turned to -90 degrees
- moved C3 51.2 mm to (134.0, 41.0), turned to 90 degrees
- moved R1 50.5 mm to (111.5, 33.2), turned to -90 degrees
- moved R4 38.4 mm to (101.0, 47.3), turned to 90 degrees
- moved U1 32.0 mm to (122.5, 37.4), turned to 180 degrees
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Connections:
- C2 pad 1: Net-(J1-Pin_3) -> Net-(J2-Pin_1)
- L1 pad 1: Net-(J1-Pin_3) -> Net-(J2-Pin_1)
- R2-2 pad 2: Net-(J1-Pin_3) -> Net-(J2-Pin_1)
- R6 pad 1: Net-(J1-Pin_9) -> Net-(J5-Pin_2)
- R7 pad 1: Net-(J1-Pin_10) -> Net-(J6-Pin_1)
- R8 pad 1: Net-(J1-Pin_8) -> Net-(J5-Pin_1)
- U3 pad J2-1: unconnected-(U3-3V3-PadJ2-1) -> Net-(J11-Pin_2)
- U3 pad J2-10: unconnected-(U3-IO26-PadJ2-10) -> Net-(U2-TX)
- U3 pad J2-11: unconnected-(U3-IO27-PadJ2-11) -> Net-(U2-RX)
- U3 pad J2-12: unconnected-(U3-IO14-PadJ2-12) -> Net-(J16-Pin_1)
- U3 pad J2-13: unconnected-(U3-IO12-PadJ2-13) -> Net-(J15-Pin_2)
- U3 pad J2-15: unconnected-(U3-IO13-PadJ2-15) -> Net-(J15-Pin_1)
- U3 pad J3-10: unconnected-(U3-IO5-PadJ3-10) -> Net-(J13-Pin_1)
- U3 pad J3-11: unconnected-(U3-IO17-PadJ3-11) -> Net-(J12-Pin_2)
- U3 pad J3-12: unconnected-(U3-IO16-PadJ3-12) -> Net-(J8-Pin_1)
- U3 pad J3-13: unconnected-(U3-IO4-PadJ3-13) -> Net-(J13-Pin_2)
- U3 pad J3-14: unconnected-(U3-IO0-PadJ3-14) -> Net-(J12-Pin_1)
- U3 pad J3-15: unconnected-(U3-IO2-PadJ3-15) -> Net-(J14-Pin_2)
- U3 pad J3-16: unconnected-(U3-IO15-PadJ3-16) -> Net-(J14-Pin_1)
- U3 pad J3-2: unconnected-(U3-IO23-PadJ3-2) -> Net-(J10-Pin_1)
- U3 pad J3-3: unconnected-(U3-IO22-PadJ3-3) -> Net-(J9-Pin_1)
- U3 pad J3-6: unconnected-(U3-IO21-PadJ3-6) -> Net-(J8-Pin_2)
- U3 pad J3-8: unconnected-(U3-IO19-PadJ3-8) -> Net-(J10-Pin_2)
- U3 pad J3-9: unconnected-(U3-IO18-PadJ3-9) -> Net-(J11-Pin_1)
Routing:
- net GNDREF: track 0.00 -> 349.3 mm, vias 0 -> 2
- net Net-(U3-IO35): track 0.00 -> 144.9 mm
- net +6V: track 0.00 -> 122.8 mm
- net Net-(U3-IO34): track 0.00 -> 111.0 mm
- net Net-(J11-Pin_2): track 0.00 -> 71.8 mm
- net Net-(J10-Pin_1): track 0.00 -> 55.6 mm
- net Net-(J11-Pin_1): track 0.00 -> 54.3 mm
- net Net-(D1-K): track 0.00 -> 51.0 mm
- net Net-(J8-Pin_2): track 0.00 -> 46.9 mm
- net Net-(J2-Pin_1): track 0.00 -> 44.8 mm
- net Net-(J8-Pin_1): track 0.00 -> 39.2 mm
- net Net-(J10-Pin_2): track 0.00 -> 39.0 mm
- net Net-(J12-Pin_2): track 0.00 -> 32.7 mm
- net Net-(J7-Pin_2): track 0.00 -> 31.8 mm
- net Net-(U2-TX): track 0.00 -> 31.6 mm
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Other:
- board outline added: 9 x 25 mm
