File: Building Resources/KiCad PCB Files/DFPlayer_LCD/DFPlayer and LCD.kicad_sch (KiCad schematic)
At the start: 2 parts, among them J1 Conn_01x06_Socket, U1 DFR0299

Commit message: More updates, finally.
Connections:
- no-connect marks 8 -> 10
Changed lines of the file:
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@@
 	(generator_version "8.0")
 	(paper "A4")
-	(junction
-		(at 153.67 86.36)
-		(diameter 0)
-		(color 0 0 0 0)
-	)
 	(no_connect
 		(at 113.03 99.06)
@@
 	(no_connect
 		(at 143.51 116.84)
+	)
+	(no_connect
+		(at 143.51 86.36)
 	)
 	(no_connect
@@
 		(at 113.03 93.98)
 	)
-	(wire
-		(pts
-			(xy 144.78 86.36) (xy 153.67 86.36)
-		)
-		(stroke
-			(width 0)
-			(type default)
-		)
+	(no_connect
+		(at 143.51 88.9)
 	)
 	(wire
@@
 	(wire
 		(pts
+			(xy 144.78 93.98) (xy 143.51 93.98)
+		)
+		(stroke
+			(width 0)
+			(type default)
+		)
+	)
+	(wire
+		(pts
 			(xy 143.51 96.52) (xy 146.05 96.52)
 		)
@@
 	(wire
 		(pts
-			(xy 154.94 86.36) (xy 153.67 86.36)
+			(xy 144.78 86.36) (xy 144.78 93.98)
 		)
 		(stroke
@@
 	(wire
 		(pts
-			(xy 144.78 86.36) (xy 144.78 93.98)
-		)
-		(stroke
-			(width 0)
-			(type default)
-		)
-	)
-	(wire
-		(pts
 			(xy 148.59 88.9) (xy 153.67 88.9)
 		)
@@
 	(wire
 		(pts
-			(xy 144.78 93.98) (xy 143.51 93.98)
+			(xy 113.03 109.22) (xy 153.67 109.22)
 		)
 		(stroke
@@
 	(wire
 		(pts
-			(xy 113.03 109.22) (xy 153.67 109.22)
+			(xy 144.78 86.36) (xy 153.67 86.36)
 		)
 		(stroke
+			(width 0)
+			(type default)
+		)
+	)
+	(wire
+		(pts
+			(xy 226.06 78.74) (xy 226.06 107.95)
+		)
+		(stroke
