File: Building Resources/KiCad PCB Files/Power_System/Power System.kicad_sch (KiCad schematic)
At the start: 15 parts, among them J1 Conn_01x02_Socket, J2 Conn_01x02_Socket, J3 Conn_01x02_Socket, J4 Conn_01x02_Socket, J5 Conn_01x02_Socket, U1 LM2596T-3.3

Commit message: Update KiCad Files
Parts:
- removed J1, J2, J3, J4, J5: Conn_01x02_Socket, Connector_PinSocket_2.54mm:PinSocket_1x02_P2.54mm_Vertical, symbol Connector:Conn_01x02_Socket
- added J1: Conn_01x10, Connector_PinSocket_2.54mm:PinSocket_1x10_P2.54mm_Vertical, symbol Connector_Generic:Conn_01x10
- C2: value 220u -> 220uF
- L1: value 68m -> 68mH
- R2-1: value 18k -> 1.6k
- R2-2: value 120k -> 1.6k
- R3: value 82k -> 1k
- U1: footprint Package_TO_SOT_THT:TO-220-5_P3.4x3.7mm_StaggerOdd_Lead3.8mm_Vertical -> LM2596TVADJG:TO170P470X1016X2092-5P
Connections:
- net +6V: now also J1.4 (Pin_4)
- net GNDREF: now also J1.10 (Pin_10), J1.3 (Pin_3), J1.8 (Pin_8), J1.9 (Pin_9)
- net at R1.2, R2.1: now also J1.1 (Pin_1)
- net at U1.5 (~{ON}/OFF): now also J1.2 (Pin_2)
- net at C2.1, L1.1, R2-2.2: now also J1.5 (Pin_5), J1.6 (Pin_6), J1.7 (Pin_7)
Other:
- note added: "GND 6V Input 3.3V Output 3.3V Output 3.3V Output GND GND GND ON/OFF Signal State of Charge Signal"
- note added: "Power Delivery Sub-Project"

Commit message: More updates, finally.
Parts:
- removed R2-2: 1.6k, Resistor_THT:R_Axial_DIN0207_L6.3mm_D2.5mm_P7.62mm_Horizontal, symbol Device:R
Connections:
- net at R2-1.2: now also C2.1, J1.5 (Pin_5), J1.6 (Pin_6), J1.7 (Pin_7), L1.1
Other:
- note removed: "Power Delivery Sub-Project"
Changed lines of the file:
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@@
 	(wire
 		(pts
-			(xy 146.05 62.23) (xy 146.05 63.5)
+			(xy 146.05 54.61) (xy 146.05 63.5)
 		)
 		(stroke
@@
 	)
 	(rectangle
-		(start 76.2 26.67)
+		(start 76.2 25.4)
 		(end 205.74 90.17)
 		(stroke
@@
 		)
 	)
-	(text "Power Delivery Sub-Project"
-		(exclude_from_sim no)
-		(at 104.902 29.718 0)
-		(effects
-			(font
-				(size 2.54 2.54)
-			)
-		)
-	)
 	(text "GND\n6V Input\n3.3V Output\n3.3V Output\n3.3V Output\nGND\nGND\nGND\nON/OFF Signal\nState of Charge \nSignal"
 		(exclude_from_sim no)
-		(at 183.388 48.514 0)
+		(at 182.372 42.926 0)
 		(effects
 			(font
@@
 				)
 				(justify left)
+				(hide yes)
 			)
 		)
@@
 					(unit 1)
 				)
-			)
-		)
-	)
-	(symbol
-		(lib_id "Device:R")
-		(at 146.05 58.42 0)
-		(unit 1)
-		(exclude_from_sim no)
-		(in_bom yes)
-		(on_board yes)
-		(dnp no)
-		(property "Reference" "R2-2"
-			(at 144.018 61.214 90)
-			(effects
-				(font
-					(size 1.27 1.27)
-				)
-				(justify left)
-			)
-		)
-		(property "Value" "1.6k"
-			(at 146.05 60.706 90)
-			(effects
-				(font
-					(size 1.27 1.27)
-				)
-				(justify left)
-			)
-		)
-		(property "Footprint" "Resistor_THT:R_Axial_DIN0207_L6.3mm_D2.5mm_P7.62mm_Horizontal"
-			(at 144.272 58.42 90)
-			(effects
-				(font
-					(size 1.27 1.27)
-				)
-				(hide yes)
-			)
-		)
-		(property "Datasheet" "~"
-			(at 146.05 58.42 0)
-			(effects
-				(font
-					(size 1.27 1.27)
-				)
-				(hide yes)
-			)
-		)
-		(property "Description" "Resistor"
-			(at 146.05 58.42 0)
-			(effects
-				(font
-					(size 1.27 1.27)
-				)
-				(hide yes)
-			)
-		)
-		(pin "1"
-		)
-		(pin "2"
-		)
-		(instances
-			(project "Power System"
-				(path "/f9f56fcb-638a-40d4-be6c-886cde0af03d"
-					(reference "R2-2")
-					(unit 1)
-				)
